File: PCB-design/cvt-hmi_22-23.kicad_sch (KiCad schematic)
At the start: 11 parts, among them IC1 LD1117V50, J1 12V Supply, J2 16x4 LCD I2C, SW1 HMI contr.

Commit message: Added some footprint assignments
Parts:
- added J2: Wheel_Hall, symbol Connector_Generic:Conn_01x01
- renumbered J2 to J3
Connections:
- net Wheel_Hall: no longer names the net of R1.1
- net Wheel_Hall: now also J2.1 (Pin_1)
Other:
- note added: "Kan behöva ändra storlek på kondensator, behöver mäta spänningsfall och tidsintervall för att veta."
- moved on the sheet: C3, J3, R1, R2, SW1
